File: DDR3_SODIMM/DDR3_SODIMM.sch (KiCad schematic (older format))
At the start: 96 parts, among them U1 DDR3_SODIMM_PINOUT

Commit message: UPD
Connections:
- net EVENT_n: no longer names the net of U?.7 (EVENT)
- no-connect marks 0 -> 1
Changed lines of the file:
@@
 EESchema Schematic File Version 4
-LIBS:DDR3_SODIMM-cache
 EELAYER 30 0
 EELAYER END
@@
 Text GLabel 15500 9000 2    50   Input ~ 0
 SA2
-Text GLabel 15500 9150 2    50   Input ~ 0
-EVENT_n
-Wire Wire Line
-	15500 9150 15250 9150
 Wire Wire Line
 	15250 9000 15500 9000
@@
 Text Notes 14250 7900 2    118  ~ 24
 TEMPERATURE
+NoConn ~ 15250 9150
 $EndSCHEMATC
